File: audio.kicad_sch (KiCad schematic)
At the start: 29 parts, among them J16 SPEAKER, J17 SPEAKER, U10 TLV320AIC3100, Y2 12.0M

Commit message: Complete Mouser part numbers for Rev C
Parts:
- C39, C42: PN (none) -> 603-CC402JRNPO9BN471
- C40, C41, C43, C45: PN (none) -> 187-CL05A105KA5NQNC
- R27, R52: PN (none) -> 303-0402WGF2001TCE
- R54: PN (none) -> 303-0402WGF1003TCE
- U10: PN (none) -> 595-V320AIC3100IRHBR
- Y2: MPN 520-2520MV-120-BN-T -> ECS-2520MV-120-BN-TR; PN (none) -> 520-2520MV-120-BN-T
