File: connectors.kicad_sch (KiCad schematic)
At the start: 24 parts, among them J12 USB_C, J13 2.5mm, J14 3.5mm, J3 GND spring, SW2 10k, U8 USBLC6-2SC6

Commit message: Complete Mouser part numbers for Rev C
Parts:
- R3: PN (none) -> 303-0402WGF1003TCE
- R46, R47: PN (none) -> 303-0402WGF5101TCE
- R48: PN (none) -> 303-0402WGF1001TCE
- R49: PN (none) -> 303-0402WGF1502TCE
- R50, R51: PN (none) -> 303-0402WGF1000TCE
