File: display.kicad_sch (KiCad schematic)
At the start: 17 parts, among them J5 LCD, Q3 BSS138, Q4 BSS138

Commit message: Complete Mouser part numbers for Rev C
Parts:
- D4: value LED -> LED Red; LCSC C25503345 -> (none); MPN XL-1005SURC -> SM0402RC; PN (none) -> 749-SM0402RC
- D5: value LED -> LED Green; LCSC C965793 -> (none); MPN XL-1005UGC -> SM0402GC; PN (none) -> 749-SM0402GC
- R15, R16, R33, R38: PN (none) -> 303-0402WGF1000TCE
- R34, R36: PN (none) -> 303-0402WGF1002TCE
- R35, R39: PN (none) -> 303-0402WGF4702TCE
- R37: PN (none) -> 303-0402WGF100JTCE
- R42: PN (none) -> 303-0402WGF1500TCE
