File: gnss.kicad_sch (KiCad schematic)
At the start: 15 parts, among them J4 Conn_Coaxial, U13 LG77L

Commit message: Complete Mouser part numbers for Rev C
Parts:
- C91, C92: PN (none) -> 81-GRM1555C1H101JA1D
- R17: PN (none) -> 303-0402WGF0000TCE
