File: keyboard.kicad_sch (KiCad schematic)
At the start: 10 parts, among them J10 GND, J11 Keyboard, J6 GND, J7 GND, J8 PTT, J9 BTN_2, Q5 BSS138

Commit message: Complete Mouser part numbers for Rev C
Parts:
- J11: LCSC C262665 -> (none); MPN AFC01-S16FCA-00 -> FH12-16S-0.5SH(55); PN (none) -> 798-FH12-16S-05SH55
- R43: PN (none) -> 667-ERJ-PA2F1500X
- R44: PN (none) -> 303-0402WGF4702TCE
- R45: PN (none) -> 303-0402WGF1000TCE
Changed lines of the file:
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@@
 			)
 		)
-		(property "PN" ""
+		(property "PN" "303-0402WGF4702TCE"
 			(at 165.1 101.6 0)
 			(hide yes)
@@
 		)
 		(property "MPN" "0402WGF4702TCE"
+			(at 165.1 101.6 0)
+			(hide yes)
+			(show_name no)
+			(do_not_autoplace no)
+			(effects
+				(font
+					(size 1.27 1.27)
+				)
+			)
+		)
+		(property "Mouser" ""
+			(at 165.1 101.6 0)
+			(hide yes)
+			(show_name no)
+			(do_not_autoplace no)
+			(effects
+				(font
+					(size 1.27 1.27)
+				)
+			)
+		)
+		(property "Mouser Part Number" ""
 			(at 165.1 101.6 0)
 			(hide yes)
@@
 			)
 		)
+		(property "Mouser" ""
+			(at 55.88 114.3 0)
+			(hide yes)
+			(show_name no)
+			(do_not_autoplace no)
+			(effects
+				(font
+					(size 1.27 1.27)
+				)
+			)
+		)
+		(property "Mouser Part Number" ""
+			(at 55.88 114.3 0)
+			(hide yes)
+			(show_name no)
+			(do_not_autoplace no)
+			(effects
+				(font
+					(size 1.27 1.27)
+				)
+			)
+		)
 		(pin "1"
 		)
@@
 		)
 		(property "LCSC Part" ""
+			(at 55.88 118.11 0)
+			(hide yes)
+			(show_name no)
+			(do_not_autoplace no)
+			(effects
+				(font
+					(size 1.27 1.27)
+				)
+			)
+		)
+		(property "Mouser" ""
+			(at 55.88 118.11 0)
+			(hide yes)
+			(show_name no)
+			(do_not_autoplace no)
+			(effects
+				(font
+					(size 1.27 1.27)
+				)
+			)
+		)
+		(property "Mouser Part Number" ""
 			(at 55.88 118.11 0)
 			(hide yes)
@@
 			)
 		)
-		(property "PN" ""
+		(property "PN" "667-ERJ-PA2F1500X"
 			(at 154.94 83.82 0)
 			(hide yes)
@@
 		)
 		(property "MPN" "ERJPA2F1500X"
+			(at 154.94 83.82 0)
+			(hide yes)
+			(show_name no)
+			(do_not_autoplace no)
+			(effects
+				(font
+					(size 1.27 1.27)
+				)
+			)
+		)
+		(property "Mouser" ""
+			(at 154.94 83.82 0)
+			(hide yes)
+			(show_name no)
+			(do_not_autoplace no)
+			(effects
+				(font
+					(size 1.27 1.27)
+				)
+			)
+		)
+		(property "Mouser Part Number" ""
 			(at 154.94 83.82 0)
 			(hide yes)
@@
 			)
 		)
-		(property "PN" ""
+		(property "PN" "303-0402WGF1000TCE"
 			(at 171.45 95.25 90)
 			(hide yes)
@@
 		)
 		(property "MPN" "0402WGF1000TCE"
+			(at 171.45 95.25 90)
+			(hide yes)
+			(show_name no)
+			(do_not_autoplace no)
+			(effects
+				(font
+					(size 1.27 1.27)
+				)
+			)
+		)
+		(property "Mouser" ""
+			(at 171.45 95.25 90)
+			(hide yes)
+			(show_name no)
+			(do_not_autoplace no)
+			(effects
+				(font
+					(size 1.27 1.27)
+				)
+			)
+		)
+		(property "Mouser Part Number" ""
 			(at 171.45 95.25 90)
 			(hide yes)
@@
 			)
 		)
+		(property "Mouser" ""
+			(at 55.88 110.49 0)
+			(hide yes)
+			(show_name no)
+			(do_not_autoplace no)
+			(effects
+				(font
+					(size 1.27 1.27)
+				)
+			)
+		)
+		(property "Mouser Part Number" ""
+			(at 55.88 110.49 0)
+			(hide yes)
+			(show_name no)
+			(do_not_autoplace no)
+			(effects
+				(font
+					(size 1.27 1.27)
+				)
+			)
+		)
 		(pin "1"
 		)
@@
 		)
 		(property "LCSC Part" ""
+			(at 55.88 100.33 0)
+			(hide yes)
+			(show_name no)
+			(do_not_autoplace no)
+			(effects
+				(font
+					(size 1.27 1.27)
+				)
+			)
+		)
+		(property "Mouser" ""
+			(at 55.88 100.33 0)
+			(hide yes)
+			(show_name no)
+			(do_not_autoplace no)
+			(effects
+				(font
+					(size 1.27 1.27)
+				)
+			)
+		)
+		(property "Mouser Part Number" ""
 			(at 55.88 100.33 0)
 			(hide yes)
@@
 			)
 		)
-		(property "Description" "Generic connectable mounting pin connector, single row, 01x16, script generated (kicad-library-utils/schlib/autogen/connector/)"
+		(property "Description" "16-position 0.5 mm pitch bottom-contact ZIF FFC/FPC connector, 2.0 mm height"
 			(at 123.19 92.71 0)
 			(hide yes)
@@
 			)
 		)
-		(property "PN" ""
+		(property "PN" "798-FH12-16S-05SH55"
 			(at 123.19 92.71 0)
 			(hide yes)
@@
 			)
 		)
-		(property "MPN" "AFC01-S16FCA-00"
+		(property "MPN" "FH12-16S-0.5SH(55)"
 			(at 123.19 92.71 0)
 			(hide yes)
@@
 			)
 		)
-		(property "LCSC" "C262665"
+		(property "LCSC" ""
 			(at 123.19 92.71 0)
 			(hide yes)
@@
 		)
 		(property "LCSC Part" ""
+			(at 123.19 92.71 0)
+			(hide yes)
+			(show_name no)
+			(do_not_autoplace no)
+			(effects
+				(font
+					(size 1.27 1.27)
+				)
+			)
+		)
+		(property "Mouser" ""
+			(at 123.19 92.71 0)
+			(hide yes)
+			(show_name no)
+			(do_not_autoplace no)
+			(effects
+				(font
+					(size 1.27 1.27)
+				)
+			)
+		)
+		(property "Mouser Part Number" ""
 			(at 123.19 92.71 0)
 			(hide yes)
@@
 		)
 		(property "LCSC Part" ""
+			(at 55.88 104.14 0)
+			(hide yes)
+			(show_name no)
+			(do_not_autoplace no)
+			(effects
+				(font
+					(size 1.27 1.27)
+				)
+			)
+		)
+		(property "Mouser" ""
+			(at 55.88 104.14 0)
+			(hide yes)
+			(show_name no)
+			(do_not_autoplace no)
+			(effects
+				(font
+					(size 1.27 1.27)
+				)
+			)
+		)
+		(property "Mouser Part Number" ""
 			(at 55.88 104.14 0)
 			(hide yes)
@@
 			(at 157.48 95.25 0)
 			(hide yes)
+			(show_name no)
+			(do_not_autoplace no)
+			(effects
+				(font
+					(size 1.27 1.27)
+				)
+			)
+		)
+		(property "Mouser" ""
+			(at 157.48 95.25 0)
+			(hide yes)
+			(show_name no)
+			(do_not_autoplace no)
+			(effects
+				(font
+					(size 1.27 1.27)
+				)
+			)
+		)
+		(property "Mouser Part Number" ""
+			(at 157.48 95.25 0)
+			(hide yes)
