File: mux.kicad_sch (KiCad schematic)
At the start: 7 parts, among them U4 74AHC1G126, U5 74AHC1G126

Commit message: Complete Mouser part numbers for Rev C
Parts:
- R33: PN (none) -> 303-0402WGF1000TCE
- R34: PN (none) -> 303-0402WGF1002TCE
- R35: PN (none) -> 303-0402WGF4702TCE
Changed lines of the file:
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@@
+			)
+		)
+		(property "PN" "303-0402WGF4702TCE"
+			(at 153.67 119.38 0)
+			(effects
+				(font
+					(size 1.27 1.27)
+				)
+				(hide yes)
 			)
 		)
@@
 			)
 		)
+		(property "PN" "303-0402WGF1000TCE"
+			(at 143.51 59.69 0)
+			(effects
+				(font
+					(size 1.27 1.27)
+				)
+				(hide yes)
+			)
+		)
 		(pin "1"
 		)
@@
 			(at 143.51 101.6 0)
 			(effects
+				(font
+					(size 1.27 1.27)
+				)
+				(hide yes)
+			)
+		)
+		(property "PN" "303-0402WGF1002TCE"
+			(at 143.51 101.6 0)
+			(effects
