File: power.kicad_sch (KiCad schematic)
At the start: 72 parts, among them J2 2S Battery, U12 BQ25792RQMR, U14 ATtiny826, U3 TPS565242, U4 TPS562203, U5 MCP1703Ax-330xxTT, U6 TLV74018PDBVR

Commit message: Complete Mouser part numbers for Rev C
Parts:
- C68, C69: PN (none) -> 187-CL05B473KO5NNNC
- R13, R18, R65, R67: PN (none) -> 303-0402WGF1003TCE
- R14: PN (none) -> 303-0402WGF1001TCE
- R21: PN (none) -> 303-0402WGF2203TCE
- R22, R24: PN (none) -> 303-0402WGF3002TCE
- R23: LCSC C2998045 -> (none); MPN FRC0402F1333TS -> RC0402FR-07133KL; PN (none) -> 603-RC0402FR-07133KL
- R63: PN (none) -> 303-0402WGF1000TCE
- R64: PN (none) -> 303-0402WGF6041TCE
- R66: PN (none) -> 303-0402WGF1273TCE
- R68: PN (none) -> 303-0402WGF5231TCE
- R69: PN (none) -> 303-0402WGF3012TCE
- R70: PN (none) -> 303-0402WGF1002TCE
- U14: PN (none) -> 579-ATTINY826-MU
