File: rf.kicad_sch (KiCad schematic)
At the start: 64 parts, among them IC1 SX1255IWLTRT, J1 Antenna, Q1 SI23333, Q2 BSS138, Q6 BSS138, U11 PE4312, U2 PE4312, U7 GRF5604, U9 SKY13330-397LF, Y1 32MHz

Commit message: Complete Mouser part numbers for Rev C
Parts:
- C14, C55: PN (none) -> 81-GRM1555C1H101JA1D
- C52, C54, C56: PN (none) -> 81-GJM1555C1H330FB1D
- C58: MPN (none) -> GJM1555C1H6R8BB01D; PN (none) -> 81-GJM1555C1H6R8BB1D
- C67: MPN (none) -> GJM1555C1H3R0BB01D; PN (none) -> 81-GJM1555C1H3R0BB01
- IC1: Mouser Part Number 947-SX1255IWLTRT -> (none)
- L5: MP 0402HP-20NXGRW -> (none); MPN (none) -> 0402HP-20NXGRW; Mouser 994-0402HP-20NXGRW -> (none); PN (none) -> 994-0402HP-20NXGRW
- L6: MPN (none) -> XR0908SQ-23NJLC
- L7: MPN (none) -> LQW18AN2N4C8ZD; PN (none) -> 81-LQW18AN2N4C8ZD
- L8: MPN (none) -> LQG15HH10NJ02D; PN (none) -> 81-LQG15HH10NJ02D
- Q1: PN (none) -> 78-SI2333DDS-T1-BE3
- R10, R11, R5, R6, R7, R8, R9: PN (none) -> 303-0402WGF1000TCE
- R12, R19, R20, R30, R4, R55, R56, R58, R59, R62: PN (none) -> 303-0402WGF1003TCE
- R28: MPN (none) -> 0402WGF1961TCE; PN (none) -> 303-0402WGF1961TCE
- R29: MPN (none) -> 0402WGF6041TCE; PN (none) -> 303-0402WGF6041TCE
- R31: PN (none) -> 303-0402WGF2202TCE
- U9: PN (none) -> 873-SKY13330-397LF
